File: rak3172.kicad_sch (KiCad schematic)
At the start: 1 part

Commit message: routing done, untidy
Parts:
- added ANT1: 915MHz, TestPoint:TestPoint_THTPad_D2.0mm_Drill1.0mm, symbol Device:Antenna
- added ANT2: U.FL, Connector_Coaxial:U.FL_Hirose_U.FL-R-SMT-1_Vertical, symbol Device:Antenna
- added BAT1, BAT2: 1.25mm Push-Pull 1x2, Connector_Molex:Molex_PicoBlade_53048-0210_1x02_P1.25mm_Horizontal, symbol Connector_Generic:Conn_01x02
- added BZ1: MLT-8530, LokapinLib:MagneticBuzzer_8530_SMD, symbol Device:Buzzer
- added C1, C2: C, Capacitor_SMD:C_0402_1005Metric, symbol Ai-Thinker RA-08:C
- added C10, C11, C22, C23, C33, C7: 1u, Capacitor_SMD:C_0402_1005Metric, symbol Ai-Thinker RA-08:C
- added C12, C14, C19, C24: 4.7u, Capacitor_SMD:C_0402_1005Metric, symbol Ai-Thinker RA-08:C
- added C13: 470n, Capacitor_SMD:C_0402_1005Metric, symbol Ai-Thinker RA-08:C
- added C16, C18, C20, C21, C26, C27, C28, C3, C30, C31, C4, C5, C6, C8, C9: 100n, Capacitor_SMD:C_0402_1005Metric, symbol Ai-Thinker RA-08:C
- added C17, C32: 47u, Capacitor_Tantalum_SMD:CP_EIA-3216-18_Kemet-A, symbol Device:C_Polarized_Small_US
- added C29: 10u, Capacitor_SMD:C_0402_1005Metric, symbol Ai-Thinker RA-08:C
- added D1: RED, LED_SMD:LED_0603_1608Metric, symbol Device:LED
- added D2: GREEN, LED_SMD:LED_0603_1608Metric, symbol Device:LED
- added D3: BAS516, Diode_SMD:D_SOD-523, symbol Diode:BAS516
- added DEBUG1: 1.25mm 1x5, Connector_Hirose:Hirose_DF13-05P-1.25DSA_1x05_P1.25mm_Vertical, symbol Connector_Generic:Conn_01x05
- added L1: L, Inductor_SMD:L_0402_1005Metric, symbol Device:L
- added L2: 15u, Inductor_SMD:L_0805_2012Metric, symbol Device:L
- added Q1: AO3401, Package_TO_SOT_SMD:SOT-23, symbol Device:Q_PMOS_GDS
- added Q2: SI2302, Package_TO_SOT_SMD:SOT-23, symbol Transistor_FET:TSM2302CX
- added R1, R10, R5, R7: DNP, Resistor_SMD:R_0402_1005Metric, symbol Device:R
- added R11, R15: 10k, Resistor_SMD:R_0402_1005Metric, symbol Device:R
- added R12, R13, R14: 0R, Resistor_SMD:R_0402_1005Metric, symbol Device:R
- added R16, R18, R3, R6, R8, R9: 1k, Resistor_SMD:R_0402_1005Metric, symbol Device:R
- added R17, R19, R2, R4: 100k, Resistor_SMD:R_0402_1005Metric, symbol Device:R
- added SW1, SW2: SW_Push, LokapinLib:5.2mm x 3.35mm Tactile Switch, symbol LokapinLib:SW_Push
- added TP1, TP2, TP5: TestPoint_Alt, TestPoint:TestPoint_Pad_D1.0mm, symbol Connector:TestPoint_Alt
- added TP10, TP11, TP6, TP7, TP8, TP9: TestPoint_Small, TestPoint:TestPoint_Pad_D1.0mm, symbol Connector:TestPoint_Small
- added U1: AP6683, Package_DFN_QFN:OnSemi_XDFN4-1EP_1.0x1.0mm_EP0.52x0.52mm, symbol Ai-Thinker RA-08:AP6683
- added U3: TP733xx, Package_DFN_QFN:OnSemi_XDFN4-1EP_1.0x1.0mm_EP0.52x0.52mm, symbol Ai-Thinker RA-08:TP733xx
- added U4: UHE4913, Package_TO_SOT_SMD:SOT-23, symbol Sensor_Magnetic:SM351LT
- added U5: QMC6308, LokapinLib:QMC6308, symbol LokapinLib:QMC6308
- added U6: L80RE-M37, XCVR_L80RE-M37, symbol LokapinLib:L80RE-M37
- added U7: QMI8658, LokapinLib:QMI8658, symbol LokapinLib:QMI8658
- gave numbers to parts that had none: 1
Connections:
- net SWDIO: now reaches U2.1 (SWDIO/A9)
- net SWDIO: now also DEBUG1.3 (Pin_3)
- net VFBSMPS: now reaches U2.10 (VFBSMPS)
- net VFBSMPS: now also C13.1, C16.1, L2.2, TP5.1
- net +3V3: now reaches U2.11 (VDDMPS)
- net +3V3: now also U2.3 (VDD), U2.4 (VBAT), U2.53 (VDD_RFPA), U2.54 (VDD_RF), U2.55 (VDD), U2.6 (VREF+), U2.7 (VDDA), BZ1.1 (-), C10.1, C11.1, C12.1, C14.1, C17.1, C18.1, C19.1, C20.1, C21.1, C22.1, C23.1, C24.1, C26.1, C27.1, C30.1, C31.1, C33.1, C8.1, C9.1, D3.1 (K), DEBUG1.5 (Pin_5), Q1.3 (S), R1.1, R11.1, R15.1, R17.2, R4.1, R5.1, R7.1, SW2.1, U3.1 (VOUT), U4.1 (VCC), U5.B1 (VDD), U6.5 (V_BCKP), U7.5 (VDDIO), U7.8 (VDD)
- net GND: now reaches U2.12 (GND)
- net GND: now also U2.28 (GND), U2.35 (GND), U2.36 (GND), U2.38 (GND), U2.39 (GND), U2.46 (GND), U2.47 (GND), U2.52 (GND), U2.56 (GND), U2.65 (GND), U2.66 (GND), U2.67 (GND), U2.68 (GND), U2.69 (GND), U2.70 (GND), U2.71 (GND), U2.72 (GND), U2.73 (GND), ANT2.2 (GND), C1.2, C10.2, C11.2, C12.2, C13.2, C14.2, C16.2, C17.2, C18.2, C19.2, C2.2, C20.2, C21.2, C22.2, C23.2, C24.2, C26.2, C27.2, C28.2, C29.2, C30.2, C31.2, C32.2, C33.2, C4.2, C5.2, C6.2, C7.2, C8.2, C9.2, D1.1 (K), D2.1 (K), DEBUG1.1 (Pin_1), Q2.2 (S), R10.1, R19.2, R2.2, SW1.1, U1.4 (VM), U3.2 (GND), U4.3 (GND), U5.A1 (GND), U6.12 (GND), U6.3 (GND), U7.6 (GND), U7.7 (GND)
- net VLXSMPS: now reaches U2.13 (VLXSMPS)
- net VLXSMPS: now also L2.1
- net IMU_INT2: now reaches U2.14 (PB3/A2/SPI1_SCK/WKUP3)
- net IMU_INT2: now also U7.9 (INT2)
- net GPS_RX: now reaches U2.17 (PB6/UART1_TX)
- net GPS_RX: now also R9.1
- net GPS_TX: now reaches U2.18 (PB7/UART1_RX)
- net GPS_TX: now also R8.1
- net 1PPS: now reaches U2.19 (I2C1_SCL/PB8)
- net 1PPS: now also U6.6 (1PPS)
- net SWCLK: now reaches U2.2 (SWCLK/A10)
- net SWCLK: now also DEBUG1.2 (Pin_2)
- net IMU_INT1: now reaches U2.27 (PC6)
- net IMU_INT1: now also U7.4 (INT1)
- net at U2.29 (PA2/UART2_TX): now also TP2.1
- net at U2.30 (PA3/UART2_RX): now also TP1.1
- net RF: now reaches U2.37 (RF)
- net RF: now also C2.1, L1.1
- net BOOT0: now reaches U2.43 (BOOT0)
- net BOOT0: now also C4.1, R1.2, R2.1, SW2.3
- net NRST: now reaches U2.44 (NRST)
- net NRST: now also C6.1, DEBUG1.4 (Pin_4), R4.2, SW1.3
- net CBR_SW: now reaches U2.5 (PC13/WKUP2)
- net CBR_SW: now also R7.2, U4.2 (OUTPUT)
- net IMU_CS: now reaches U2.59 (SPI2_NSS/PB12)
- net IMU_CS: now also TP8.1, U7.12 (CS)
- net IMU_SCK: now reaches U2.60 (A0/SPI2_SCK/PB13)
- net IMU_SCK: now also R12.1, TP9.1
- net IMU_SDO: now reaches U2.61 (A1/SPI2_MISO/PB14)
- net IMU_SDO: now also R14.1, TP11.1
- net IMU_SDI: now reaches U2.62 (PA10/SPI2_MOSI)
- net IMU_SDI: now also R13.1, TP10.1
- net BUZZER: now reaches U2.63 (PA11/I2C2_SDA/A7)
- net BUZZER: now also R18.1
- net Gate_GPS: now reaches U2.64 (PA12/I2C2_SCL/A8)
- net Gate_GPS: now also R16.1
- net VBAT_SENSE: now reaches U2.8 (PA15/I2C2_SDA/A11)
- net VBAT_SENSE: now also R3.2
- net LED: now reaches U2.9 (SPI2_MOSI/PB15)
- net LED: now also R6.1
- new net: D1.2 (A), R5.2
- new net: D2.2 (A), R6.2
- new net: Q2.1 (G), R18.2, R19.1
- new net +BATT: BAT1.1 (Pin_1), BAT2.2 (Pin_2), C3.1, C5.1, C7.1, R3.1, U1.1 (VDD), U3.3 (EN), U3.4 (VIN)
- new net -BATT: BAT1.2 (Pin_2), BAT2.1 (Pin_1), C3.2, U1.2 (VSS), U1.3 (VSS)
- new net ANTENNA: ANT1.1 (A), ANT2.1 (A), C1.1, L1.2
- new net BUZZER-: BZ1.2 (+), D3.2 (A), Q2.3 (D)
- new net GPS_VDD: C28.1, C29.1, C32.1, Q1.2 (D), U6.10 (RESET), U6.4 (VCC)
- new net IMU_SCK_P: R12.2, U7.13 (SCL/SPC)
- new net IMU_SDI_P: R13.2, U7.14 (SDA/SDI/SDIO)
- new net IMU_SDO_P: R14.2, U7.1 (SDO/SA0)
- new net Magneto_SCL: R15.2, TP7.1, U5.A2 (SCL), U7.3 (MSCL)
- new net Magneto_SDA: R11.2, TP6.1, U5.B2 (SDA), U7.2 (MSDA)
- new net Q2_G: Q1.1 (G), R16.2, R17.1
- new net p_GPS_RX: R10.2, R9.2, U6.1 (RXD1)
- new net p_GPS_TX: R8.2, U6.2 (TXD1)
- no-connect marks 0 -> 20
Other:
- note added: "From https://chemandy.com/calculators/coplanar-waveguide-with-ground-calculator.htm Er = 4.6, Eeff = 3.478, track width = 0.38mm, gnd clearance = 0.4mm, thickness = 0.2mm"
- note added: "Using Grounded Coplanar Wave Guide"
- note added: "With Via Fencing, D = x mils"

Commit message: Added 3D Models (-Antenna) Added Manufacturing File (BOM/POS/Gerber) Tidied up silkscreen placement Added via stitching Added via fencing for GCPW Changed bat connector position and package (to SMD)
Parts:
- BAT1, BAT2: footprint Connector_Molex:Molex_PicoBlade_53048-0210_1x02_P1.25mm_Horizontal -> LokapinLib:1.25-2PWB DEALON
- R5: value DNP -> 1k
Changed lines of the file:
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@@
       (effects (font (size 1.27 1.27)) hide)
     )
-    (property "Datasheet" "~" (id 3) (at 114.935 113.03 0)
+    (property "Datasheet" "https://www.lcsc.com/product-detail/Inductors-SMD_microgate-MGFL2012F150MT-LF_C486333.html" (id 3) (at 114.935 113.03 0)
       (effects (font (size 1.27 1.27)) hide)
     )
@@
     (property "Reference" "BAT2" (id 0) (at 35.56 27.94 0))
     (property "Value" "1.25mm Push-Pull 1x2" (id 1) (at 31.75 29.845 0))
-    (property "Footprint" "Connector_Molex:Molex_PicoBlade_53048-0210_1x02_P1.25mm_Horizontal" (id 2) (at 35.56 36.195 0)
-      (effects (font (size 1.27 1.27)) hide)
-    )
-    (property "Datasheet" "https://www.lcsc.com/product-detail/Wire-To-Board-Wire-To-Wire-Connector_HCTL-HC-1-25-2AW_C2845535.html" (id 3) (at 35.56 36.195 0)
+    (property "Footprint" "LokapinLib:1.25-2PWB DEALON" (id 2) (at 35.56 36.195 0)
+      (effects (font (size 1.27 1.27)) hide)
+    )
+    (property "Datasheet" "https://www.lcsc.com/product-detail/Wire-To-Board-Wire-To-Wire-Connector_DEALON-1-25-2PWB_C2905009.html" (id 3) (at 35.56 36.195 0)
       (effects (font (size 1.27 1.27)) hide)
     )
@@
       (effects (font (size 1.27 1.27)) hide)
     )
-    (property "Datasheet" "~" (id 3) (at 62.23 177.165 0)
+    (property "Datasheet" "https://datasheet.lcsc.com/lcsc/2108261830_BZCN-TSA017A2518A_C2888884.pdf" (id 3) (at 62.23 177.165 0)
       (effects (font (size 1.27 1.27)) hide)
     )
@@
       (effects (font (size 1.27 1.27)) hide)
     )
-    (property "Datasheet" "~" (id 3) (at 24.13 175.26 0)
+    (property "Datasheet" "https://datasheet.lcsc.com/lcsc/2108261830_BZCN-TSA017A2518A_C2888884.pdf" (id 3) (at 24.13 175.26 0)
       (effects (font (size 1.27 1.27)) hide)
     )
@@
       (effects (font (size 1.27 1.27)) hide)
     )
-    (property "Footprint" "Connector_Molex:Molex_PicoBlade_53048-0210_1x02_P1.25mm_Horizontal" (id 2) (at 24.13 33.655 0)
-      (effects (font (size 1.27 1.27)) hide)
-    )
-    (property "Datasheet" "https://www.lcsc.com/product-detail/Wire-To-Board-Wire-To-Wire-Connector_HCTL-HC-1-25-2AW_C2845535.html" (id 3) (at 24.13 33.655 0)
+    (property "Footprint" "LokapinLib:1.25-2PWB DEALON" (id 2) (at 24.13 33.655 0)
+      (effects (font (size 1.27 1.27)) hide)
+    )
+    (property "Datasheet" "https://www.lcsc.com/product-detail/Wire-To-Board-Wire-To-Wire-Connector_DEALON-1-25-2PWB_C2905009.html" (id 3) (at 24.13 33.655 0)
       (effects (font (size 1.27 1.27)) hide)
     )
@@
       (effects (font (size 1.27 1.27)) (justify left))
     )
-    (property "Value" "DNP" (id 1) (at 88.9 177.165 0)
+    (property "Value" "1k" (id 1) (at 88.9 177.165 0)
       (effects (font (size 1.27 1.27)) (justify left))
     )
@@
     )
     (path "/87d19926-fddc-44cc-8f1c-eabeb5918bbf"
-      (reference "BAT1") (unit 1) (value "1.25mm Push-Pull 1x2") (footprint "Connector_Molex:Molex_PicoBlade_53048-0210_1x02_P1.25mm_Horizontal")
+      (reference "BAT1") (unit 1) (value "1.25mm Push-Pull 1x2") (footprint "LokapinLib:1.25-2PWB DEALON")
     )
     (path "/296fadc0-2da8-4886-8880-b52a8b6707e0"
-      (reference "BAT2") (unit 1) (value "1.25mm Push-Pull 1x2") (footprint "Connector_Molex:Molex_PicoBlade_53048-0210_1x02_P1.25mm_Horizontal")
+      (reference "BAT2") (unit 1) (value "1.25mm Push-Pull 1x2") (footprint "LokapinLib:1.25-2PWB DEALON")
     )
     (path "/04bb5b47-eb1c-4c53-8040-6071e03c7a67"
@@
     )
     (path "/99495766-53c7-4f15-90ea-bfb6bca1784c"
-      (reference "R5") (unit 1) (value "DNP") (footprint "Resistor_SMD:R_0402_1005Metric")
+      (reference "R5") (unit 1) (value "1k") (footprint "Resistor_SMD:R_0402_1005Metric")
     )
     (path "/5bdeab38-87af-4886-bbdc-7cc576377745"
